File: Kicad/MarcadorPing/MarcadorPing.kicad_sch (KiCad schematic)
At the start: 14 parts, among them J1 Conn_01x02_Male, SW1 SW_SPDT, U1 ATmega328P-P, U2 NRF24L01_Breakout, U3 TP4056, U4 AMS1117-3.3_module, Y1 Crystal

Commit message: diseño pcb
Parts:
- B1: footprint (none) -> Scoreboard:TTP223B
- J1: footprint Connector_PinHeader_2.54mm:PinHeader_1x02_P2.54mm_Horizontal -> Scoreboard:LiPo 502030
- U2: footprint RF_Module:nRF24L01_Breakout -> Scoreboard:NRF24L01
- U3: footprint (none) -> Scoreboard:TP4056
- U4: footprint (none) -> Scoreboard:AMS1117
