File: Kicad/MarcadorPing/MarcadorPing.kicad_pcb (KiCad board)
At the start: 2 copper layers, 49.3 x 100.1 mm, 14 parts, among them J1 Conn_01x02_Male, SW1 SW_SPDT, U1 ATmega328P-P, U2 NRF24L01_Breakout, U3 TP4056, U4 AMS1117-3.3_module, Y1 Crystal

Commit message: Cambios placas
Routing:
- net Net-(J1-Pin_2): track 35.0 -> 25.1 mm
- net Net-(J1-Pin_1): track 31.1 -> 21.2 mm
- net (no net): vias 0 -> 3
Changed lines of the file:
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@@
     (fp_rect (start -10.25 3) (end 10.25 35)
       (stroke (width 0.2) (type default)) (fill none) (layer "F.Mask"))
-    (pad "1" thru_hole rect (at 12.7 5.08) (size 1.8 1.8) (drill 0.3) (layers "*.Cu" "*.Mask")
+    (pad "1" thru_hole rect (at 12.7 15) (size 1.8 1.8) (drill 0.3) (layers "*.Cu" "*.Mask")
       (net 7 "Net-(J1-Pin_1)") (pinfunction "Pin_1") (pintype "passive"))
-    (pad "2" thru_hole rect (at 15.24 5.08) (size 1.8 1.8) (drill 0.3) (layers "*.Cu" "*.Mask")
+    (pad "2" thru_hole rect (at 15.24 15) (size 1.8 1.8) (drill 0.3) (layers "*.Cu" "*.Mask")
       (net 32 "Net-(J1-Pin_2)") (pinfunction "Pin_2") (pintype "passive"))
   )
@@
   (gr_rect (start 124.12 57.18) (end 173.42 157.28)
     (stroke (width 0.1) (type default)) (fill none) (layer "Edge.Cuts"))
+  (via (at 149.02 60.58) (size 2.5) (drill 2.4) (layers "F.Cu" "B.Cu") (net 0))
+  (via (at 127.12 153.98) (size 2.5) (drill 2.4) (layers "F.Cu" "B.Cu") (net 0))
+  (via (at 170.12 154.08) (size 2.5) (drill 2.4) (layers "F.Cu" "B.Cu") (net 0))
   (segment (start 138.32 136.78) (end 150.62 136.78) (width 1) (layer "B.Cu") (net 1))
   (segment (start 136.25 134.71) (end 138.32 136.78) (width 1) (layer "B.Cu") (net 1))
@@
   (segment (start 143.87 114.73) (end 145.27 114.73) (width 1) (layer "B.Cu") (net 6))
   (segment (start 157.22 81.38) (end 158.32 82.48) (width 1) (layer "B.Cu") (net 7))
-  (segment (start 147.925 61.935) (end 147.925 77.885) (width 1) (layer "B.Cu") (net 7))
+  (segment (start 147.925 77.885) (end 147.925 71.855) (width 1) (layer "B.Cu") (net 7))
   (segment (start 151.42 81.38) (end 157.22 81.38) (width 1) (layer "B.Cu") (net 7))
   (segment (start 147.925 77.885) (end 151.42 81.38) (width 1) (layer "B.Cu") (net 7))
@@
   (segment (start 141.82 133.28) (end 140.22 131.68) (width 1) (layer "B.Cu") (net 22))
   (segment (start 141.75 122.35) (end 143.87 122.35) (width 1) (layer "B.Cu") (net 22))
-  (segment (start 150.465 61.935) (end 150.465 76.625) (width 1) (layer "B.Cu") (net 32))
+  (segment (start 150.465 71.855) (end 150.465 76.625) (width 1) (layer "B.Cu") (net 32))
   (segment (start 165.32 82.18) (end 165.32 85.355) (width 1) (layer "B.Cu") (net 32))
   (segment (start 162.72 79.58) (end 165.32 82.18) (width 1) (layer "B.Cu") (net 32))
@@
         (xy 124.82 57.88)
         (xy 172.72 57.88)
-        (xy 172.52 147.88)
-        (xy 125.32 147.78)
+        (xy 172.22 156.48)
+        (xy 125.02 156.38)
       )
     )
