File: Kicad/MarcadorPing2/MarcadorPing2.kicad_pcb (KiCad board)
At the start: 2 copper layers, 90.6 x 76.8 mm, 24 parts, among them J1 Jack-DC, SW1 SW_SPST, SW2 SW_SPST, SW3 SW_Push, SW4 SW_Push, SW5 SW_Push, SW6 SW_Push, U1 NRF24L01_Breakout, U2 AMS1117-3.3_module, U3 ATmega328P-P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

Commit message: Cambios placas
Parts:
- C4, C5: footprint Capacitor_SMD:C_1206_3216Metric_Pad1.33x1.80mm_HandSolder -> Capacitor_THT:C_Disc_D3.8mm_W2.6mm_P2.50mm
Routing:
- net Net-(U3-XTAL2/PB7): track 11.7 -> 13.2 mm
- net GND: track 200.6 -> 199.1 mm
- net Net-(U3-XTAL1/PB6): track 11.8 -> 10.9 mm
- net (no net): vias 0 -> 4
Other:
- board size 90.6 x 76.8 mm -> 98 x 76.8 mm
