File: Kicad/MarcadorPing2/MarcadorPing2.kicad_sch (KiCad schematic)
At the start: 14 parts, among them J1 Jack-DC, SW1 SW_SPST, SW2 SW_SPST, SW3 SW_Push, SW4 SW_Push, SW5 SW_Push, U1 NRF24L01_Breakout, U2 AMS1117-3.3_module

Commit message: diseño pcb
Parts:
- added BZ1: Buzzer, TerminalBlock_Phoenix:TerminalBlock_Phoenix_MKDS-1,5-2_1x02_P5.00mm_Horizontal, symbol Device:Buzzer
- added C2: 100nF, Capacitor_THT:C_Disc_D3.8mm_W2.6mm_P2.50mm, symbol pspice:C
- added C3: 100nF, Capacitor_THT:C_Disc_D3.8mm_W2.6mm_P2.50mm, symbol Device:C_Small
- added C4, C5: 22pF, Capacitor_SMD:C_1206_3216Metric_Pad1.33x1.80mm_HandSolder, symbol Device:C_Small
- added R5: 10k, Resistor_THT:R_Axial_DIN0207_L6.3mm_D2.5mm_P7.62mm_Horizontal, symbol Device:R
- added R6: 100, Resistor_THT:R_Axial_DIN0207_L6.3mm_D2.5mm_P7.62mm_Horizontal, symbol Device:R
- added SW6: SW_Push, TerminalBlock_Phoenix:TerminalBlock_Phoenix_MKDS-1,5-2_1x02_P5.00mm_Horizontal, symbol Switch:SW_Push
- added U3: ATmega328P-P, Package_DIP:DIP-28_W7.62mm, symbol MCU_Microchip_ATmega:ATmega328P-P
- added Y1: Crystal, Crystal:Resonator-2Pin_W8.0mm_H3.5mm, symbol Device:Crystal
- SW1, SW2, SW3, SW4, SW5: footprint TerminalBlock:TerminalBlock_Altech_AK300-2_P5.00mm -> TerminalBlock_Phoenix:TerminalBlock_Phoenix_MKDS-1,5-2_1x02_P5.00mm_Horizontal
- U1: footprint (none) -> Scoreboard:NRF24L01
- U2: footprint (none) -> Scoreboard:AMS1117
Connections:
- net +5V: now also C2.1, R5.2, U3.20 (AVCC), U3.7 (VCC)
- net GND: now also BZ1.2 (+), C2.2, C3.1, C4.1, C5.2, SW6.1, U3.22 (GND), U3.8 (GND)
- net B-RES: now reaches A1.3 (~{RESET})
- net B-RES: now also SW6.2
- new net: R5.1, U3.1 (~{RESET}/PC6)
- new net: BZ1.1 (-), R6.2
- new net: C5.1, U3.10 (XTAL2/PB7), Y1.1
- new net: C4.2, U3.9 (XTAL1/PB6), Y1.2
- new net: C3.2, U3.21 (AREF)
- new net BUZZ: R6.1, U3.15 (PB1)
- no-connect marks 18 -> 35
Other:
- note added: "Arduino Nano"
- note added: "Atmega328p"
- note added: "Botón Reset"
- note added: "Buzzer"
- note removed: "Microcontrolador"
- moved on the sheet: C1, J1, R1, R2, R3, R4, SW1, SW2, SW3, SW4, SW5, U1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

Commit message: Cambios placas
Connections:
- no-connect marks 35 -> 36
Changed lines of the file:
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@@
   (no_connect (at 34.29 42.672))
   (no_connect (at 251.46 66.04))
+  (no_connect (at 59.69 42.672))
   (no_connect (at 59.69 70.612))
   (no_connect (at 49.53 32.512))
